File: flight/electronics/power_board.brd (EAGLE design)
At the start: 80 x 80 mm, 13 parts, among them IC1 7808T, X1 JST-XH-02-PIN, X2 JST-XH-03-PIN, X3 JST-XH-03-PIN, X4 JST-XH-02-PIN, X6 JST-XH-03-PIN

Commit message: power/sensor
Parts:
- removed H4: MOUNT-PAD-ROUND3.0, holes:3,0-PAD
- removed IC1: 7808T, linear:TO220H
- added H5: MOUNT-PAD-ROUND3.0, holes:3,0-PAD
- added U$1: LD1086V33-DG, linear:TO220H
- C1: value 0.33uF -> 33uF
- C2: value 0.1uF -> 0.47uF
- moved H3 101.8 mm to (76.0, 4.00)
- moved H2 72.0 mm to (4.00, 4.00)
- moved X3 59.9 mm to (27.6, 10.2), turned to 180 degrees
- moved X6 23.4 mm to (12.6, 68.8)
- moved C2 19.2 mm to (36.7, 10.9), turned to 180 degrees
- moved C1 19.0 mm to (36.7, 16.2), turned to 180 degrees
- moved X2 11.6 mm to (24.6, 68.8)
- moved X1 4.96 mm to (65.0, 69.9)
- moved X4 2.89 mm to (15.1, 10.2)
- moved B1 0.06 mm to (3.94, 49.5)
Connections:
- removed net N$2: H1.B3,0, H2.B3,0, H3.B3,0, H4.B3,0
- removed net N$4: B1.3
- net 3V3: now also U$1.2; no longer IC1.3
- net GND: now also B1.3, H1.B3,0, H2.B3,0, H3.B3,0, H5.B3,0, U$1.1; no longer IC1.2
- net SWO: now also U$1.3; no longer IC1.1
Routing:
- net VBAT: track 0.00 -> 147.2 mm
- net 3V3: track 0.00 -> 106.8 mm, vias 0 -> 1
- net SWO: track 0.00 -> 73.7 mm
- net N$1: track 0.00 -> 19.1 mm
- added copper zone on layer 1, net GND
- added copper zone on layer 16, net GND
Other:
- board text added: "+"
- board text added: "-"
- board text added: "BAT"
- board text added: "KAOS 1 POWER BOWRD REV1"
- board text added: "PRIME"
- board text added: "PW SWITCH"
- board text removed: "PRIM"
- board text removed: "SW"
