File: flight/electronics/sensor_board.brd (EAGLE design)
At the start: 80 x 80 mm, 9 parts, among them U1 GY-521MPU6050, X1 JST-XH-03-PIN, X2 JST-XH-07-PIN

Commit message: power/sensor
Parts:
- removed U$2, U$3, U$4, U$5: (no value), holes:3,0
- added H1, H2, H3, H4: MOUNT-PAD-ROUND3.0, holes:3,0-PAD
- added R1: therm, Resistor:RESAD1176W63L850D250B
- added R2: res, Resistor:RESAD1176W63L850D250B
- moved X2 12.9 mm to (53.9, 69.8)
- moved X1 7.44 mm to (12.6, 69.3)
- moved U$6 2.69 mm to (12.5, 11.0)
- moved U$1 2.50 mm to (12.5, 40.0)
- moved U1 1.50 mm to (63.5, 40.0)
Connections:
- net 3V3: now also R1.2
- net GND: now also H1.B3,0, H2.B3,0, H3.B3,0, H4.B3,0, R2.1
- net GPIO3: now also R1.1, R2.2
Routing:
- net 3V3: track 0.00 -> 149.5 mm
- net SCL: track 0.00 -> 87.6 mm
- net SDA: track 0.00 -> 77.9 mm, vias 0 -> 1
- net GPIO1: track 0.00 -> 71.9 mm
- net GPIO2: track 0.00 -> 43.6 mm
- net GPIO3: track 0.00 -> 37.0 mm
- added copper zone on layer 1, net GND
- added copper zone on layer 16, net GND
Other:
- board text added: "KOAS 1 Sensor Board Rev1"
- board text added: "SCD"
- board text removed: "KSC Sensor Board Rev1"
