File: flight/electronics/sensor_board.sch (EAGLE design)
At the start: 5 parts, among them U1 GY-521MPU6050, X1 JST-XH-03-PIN, X2 JST-XH-07-PIN

Commit message: power/sensor
Parts:
- added H1, H2, H3, H4: MOUNT-PAD-ROUND3.0, holes:MOUNT-PAD-ROUND3.0
- added R1: therm, Resistor:R_AXIAL-11.7MM-PITCH
- added R2: res, Resistor:R_AXIAL-11.7MM-PITCH
Connections:
- net 3V3: now also R1.2
- net GND: now also H1.MOUNT, H2.MOUNT, H3.MOUNT, H4.MOUNT, R2.1
- net GPIO3: now also R1.1, R2.2
Other:
- note removed: "add thermister"
