File: flight/electronics/CommunicationBoard.sch (EAGLE design)
At the start: 7 parts, among them J1 CONUFL001-SMD-T, X1 JST-XH-02-PIN

Commit message: final touches
Parts:
- added H5, H6, H7, H8: MOUNT-PAD-ROUND3.0, holes:MOUNT-PAD-ROUND3.0
Connections:
- removed net SIG: H1.MOUNT, H2.MOUNT, H3.MOUNT, H4.MOUNT, J1.1
- new net SIG+: H1.MOUNT, H2.MOUNT, J1.1
- new net SIG-: H3.MOUNT, H4.MOUNT, J1.2
- net GND: now also H5.MOUNT, H6.MOUNT, H7.MOUNT, H8.MOUNT; no longer J1.2
Changed lines of the file:
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@@
 <part name="H3" library="holes" library_urn="urn:adsk.eagle:library:237" deviceset="MOUNT-PAD-ROUND" device="3.0" package3d_urn="urn:adsk.eagle:package:14280/1"/>
 <part name="H4" library="holes" library_urn="urn:adsk.eagle:library:237" deviceset="MOUNT-PAD-ROUND" device="3.0" package3d_urn="urn:adsk.eagle:package:14280/1"/>
+<part name="H5" library="holes" library_urn="urn:adsk.eagle:library:237" deviceset="MOUNT-PAD-ROUND" device="3.0" package3d_urn="urn:adsk.eagle:package:14280/1"/>
+<part name="H6" library="holes" library_urn="urn:adsk.eagle:library:237" deviceset="MOUNT-PAD-ROUND" device="3.0" package3d_urn="urn:adsk.eagle:package:14280/1"/>
+<part name="H7" library="holes" library_urn="urn:adsk.eagle:library:237" deviceset="MOUNT-PAD-ROUND" device="3.0" package3d_urn="urn:adsk.eagle:package:14280/1"/>
+<part name="H8" library="holes" library_urn="urn:adsk.eagle:library:237" deviceset="MOUNT-PAD-ROUND" device="3.0" package3d_urn="urn:adsk.eagle:package:14280/1"/>
+<part name="GND1" library="supply1" library_urn="urn:adsk.eagle:library:371" deviceset="GND" device=""/>
 </parts>
 <sheets>
@@
 <attribute name="VALUE" x="15.494" y="-5.0038" size="1.778" layer="96"/>
 </instance>
+<instance part="H5" gate="G$1" x="12.7" y="-17.78" smashed="yes">
+<attribute name="NAME" x="15.494" y="-17.1958" size="1.778" layer="95"/>
+<attribute name="VALUE" x="15.494" y="-20.2438" size="1.778" layer="96"/>
+</instance>
+<instance part="H6" gate="G$1" x="12.7" y="-25.4" smashed="yes">
+<attribute name="NAME" x="15.494" y="-24.8158" size="1.778" layer="95"/>
+<attribute name="VALUE" x="15.494" y="-27.8638" size="1.778" layer="96"/>
+</instance>
+<instance part="H7" gate="G$1" x="12.7" y="-33.02" smashed="yes">
+<attribute name="NAME" x="15.494" y="-32.4358" size="1.778" layer="95"/>
+<attribute name="VALUE" x="15.494" y="-35.4838" size="1.778" layer="96"/>
+</instance>
+<instance part="H8" gate="G$1" x="12.7" y="-40.64" smashed="yes">
+<attribute name="NAME" x="15.494" y="-40.0558" size="1.778" layer="95"/>
+<attribute name="VALUE" x="15.494" y="-43.1038" size="1.778" layer="96"/>
+</instance>
+<instance part="GND1" gate="1" x="7.62" y="-45.72" smashed="yes">
+<attribute name="VALUE" x="5.08" y="-48.26" size="1.778" layer="96"/>
+</instance>
 </instances>
 <busses>
@@
 <net name="GND" class="0">
 <segment>
-<wire x1="15.24" y1="33.02" x2="-5.08" y2="33.02" width="0.1524" layer="91"/>
 <pinref part="U$1" gate="G$1" pin="GND"/>
 <pinref part="X1" gate="-1" pin="S"/>
-<pinref part="J1" gate="G$1" pin="2"/>
-<wire x1="-5.08" y1="33.02" x2="-30.48" y2="33.02" width="0.1524" layer="91"/>
-<wire x1="-7.62" y1="7.62" x2="-5.08" y2="7.62" width="0.1524" layer="91"/>
-<wire x1="-5.08" y1="7.62" x2="-5.08" y2="33.02" width="0.1524" layer="91"/>
-<junction x="-5.08" y="33.02"/>
+<wire x1="15.24" y1="33.02" x2="-30.48" y2="33.02" width="0.1524" layer="91"/>
+</segment>
+<segment>
+<pinref part="GND1" gate="1" pin="GND"/>
+<pinref part="H8" gate="G$1" pin="MOUNT"/>
+<wire x1="7.62" y1="-43.18" x2="7.62" y2="-40.64" width="0.1524" layer="91"/>
+<wire x1="7.62" y1="-40.64" x2="10.16" y2="-40.64" width="0.1524" layer="91"/>
+<pinref part="H7" gate="G$1" pin="MOUNT"/>
+<wire x1="7.62" y1="-40.64" x2="7.62" y2="-33.02" width="0.1524" layer="91"/>
+<wire x1="7.62" y1="-33.02" x2="10.16" y2="-33.02" width="0.1524" layer="91"/>
+<junction x="7.62" y="-40.64"/>
+<pinref part="H6" gate="G$1" pin="MOUNT"/>
+<wire x1="7.62" y1="-33.02" x2="7.62" y2="-25.4" width="0.1524" layer="91"/>
+<wire x1="7.62" y1="-25.4" x2="10.16" y2="-25.4" width="0.1524" layer="91"/>
+<junction x="7.62" y="-33.02"/>
+<pinref part="H5" gate="G$1" pin="MOUNT"/>
+<wire x1="7.62" y1="-25.4" x2="7.62" y2="-17.78" width="0.1524" layer="91"/>
+<wire x1="7.62" y1="-17.78" x2="10.16" y2="-17.78" width="0.1524" layer="91"/>
+<junction x="7.62" y="-25.4"/>
 </segment>
 </net>
@@
 </segment>
 </net>
-<net name="SIG" class="0">
+<net name="SIG+" class="0">
 <segment>
 <pinref part="J1" gate="G$1" pin="1"/>
@@
 <wire x1="10.16" y1="12.7" x2="5.08" y2="12.7" width="0.1524" layer="91"/>
 <junction x="5.08" y="12.7"/>
+</segment>
+</net>
+<net name="SIG-" class="0">
+<segment>
+<pinref part="J1" gate="G$1" pin="2"/>
+<wire x1="-7.62" y1="7.62" x2="5.08" y2="7.62" width="0.1524" layer="91"/>
 <pinref part="H3" gate="G$1" pin="MOUNT"/>
 <wire x1="10.16" y1="5.08" x2="5.08" y2="5.08" width="0.1524" layer="91"/>
-<wire x1="5.08" y1="5.08" x2="5.08" y2="10.16" width="0.1524" layer="91"/>
-<junction x="5.08" y="10.16"/>
 <pinref part="H4" gate="G$1" pin="MOUNT"/>
 <wire x1="10.16" y1="-2.54" x2="5.08" y2="-2.54" width="0.1524" layer="91"/>
 <wire x1="5.08" y1="-2.54" x2="5.08" y2="5.08" width="0.1524" layer="91"/>
+<wire x1="5.08" y1="7.62" x2="5.08" y2="5.08" width="0.1524" layer="91"/>
 <junction x="5.08" y="5.08"/>
 </segment>

Commit message: final board tweaks
Parts:
- X1: device Rembrandt Electronics - JST XH Connectors v1-0:JST-XH-02-PIN -> JST-XH Connectors:JST-XH-02-PIN
Changed lines of the file:
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@@
 </classes>
 <parts>
-<part name="X1" library="Rembrandt Electronics - JST XH Connectors v1-0" deviceset="JST-XH-02-PIN" device=""/>
+<part name="X1" library="JST-XH Connectors" deviceset="JST-XH-02-PIN" device=""/>
 <part name="U$1" library="Breakouts" deviceset="LIGHTAPRS" device=""/>
 <part name="J1" library="CONUFL001-SMD-T" deviceset="CONUFL001-SMD-T" device=""/>
