File: flight/electronics/SensorBoard.brd (EAGLE design)
At the start: 80 x 80 mm, 11 parts, among them U1 GY-521MPU6050, X1 JST-XH-03-PIN, X2 JST-XH-07-PIN

Commit message: rev1 changes
Parts:
- removed R2: res, Resistor:RESAD1176W63L850D250B
- removed U$1: BMP388_QT, BMP388_QT:BMP388_QT
- added U$2: BMP388BREAKOUT, Breakouts:BMP388BREAKOUT
- added X3: JST-XH-02-PIN, JST-XH Connectors:JST-XH_S2B
- R1: value therm -> 10kΩ; device Resistor:RESAD1176W63L850D250B -> rcl:0204/7
- moved R1 21.0 mm to (72.0, 65.0), turned to 0 degrees
Connections:
- net 3V3: now also U$2.3VO; no longer U$1.P$2
- net GND: now also U$2.GND, X3.PIN1; no longer R2.1, U$1.P$10, U$1.P$3, U$1.P$9
- net GPIO2: now also U$2.INT; no longer U$1.P$8
- net GPIO3: now also X3.PIN2; no longer R2.2
- net SCL: now also U$2.SCL; no longer U$1.P$4
- net SDA: now also U$2.SDA; no longer U$1.P$6
Routing:
- net GPIO3: track 37.0 -> 13.3 mm
- net GPIO2: track 43.6 -> 53.9 mm
- net GPIO1: track 71.9 -> 82.2 mm
- net 3V3: track 149.5 -> 158.8 mm
- net SCL: track 87.6 -> 85.6 mm
- net SDA: track 77.9 -> 78.3 mm, vias 1 -> 0
Other:
- board text added: "KAOS-1 SENSOR BOARD REV1"
- board text removed: "KOAS 1 Sensor Board Rev1"
- board text removed: "SCD"
