File: flight/electronics/SensorBoard.sch (EAGLE design)
At the start: 11 parts, among them U1 GY-521MPU6050, X1 JST-XH-03-PIN, X2 JST-XH-07-PIN

Commit message: rev1 changes
Parts:
- removed R2: res, Resistor:R_AXIAL-11.7MM-PITCH
- removed U$1: BMP388_QT, BMP388_QT:BMP388_QT
- added U$2: BMP388BREAKOUT, Breakouts:BMP388BREAKOUT
- added X3: JST-XH-02-PIN, JST-XH Connectors:JST-XH-02-PIN
- R1: value therm -> 10kΩ; device Resistor:R_AXIAL-11.7MM-PITCH -> rcl:R-US_0204/7
Connections:
- net 3V3: now also U$2.3VO; no longer U$1.3VO
- net GND: now also U$2.GND, X3-1.S; no longer R2.1, U$1.GND
- net GPIO2: now also U$2.INT; no longer U$1.INT
- net GPIO3: now also X3-2.S; no longer R2.2
- net SCL: now also U$2.SCL; no longer U$1.SCL
- net SDA: now also U$2.SDA; no longer U$1.SDI
Other:
- note removed: "double check these pins"
Changed lines of the file:
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@@
 <parts>
 <part name="FRAME1" library="frames" library_urn="urn:adsk.eagle:library:229" deviceset="A4L-LOC" device=""/>
-<part name="U$1" library="BMP388_QT" deviceset="BMP388_QT" device=""/>
-<part name="SUPPLY1" library="supply2" library_urn="urn:adsk.eagle:library:372" deviceset="GND" device=""/>
 <part name="SUPPLY2" library="supply2" library_urn="urn:adsk.eagle:library:372" deviceset="GND" device=""/>
 <part name="SUPPLY3" library="supply2" library_urn="urn:adsk.eagle:library:372" deviceset="GND" device=""/>
@@
 <part name="U1" library="GY-521" deviceset="GY-521" device="MPU6050"/>
 <part name="X2" library="JST-XH Connectors" deviceset="JST-XH-07-PIN" device=""/>
-<part name="R1" library="Resistor" library_urn="urn:adsk.eagle:library:16378527" deviceset="R" device="AXIAL-11.7MM-PITCH" package3d_urn="urn:adsk.eagle:package:16378560/2" technology="_" value="therm"/>
-<part name="R2" library="Resistor" library_urn="urn:adsk.eagle:library:16378527" deviceset="R" device="AXIAL-11.7MM-PITCH" package3d_urn="urn:adsk.eagle:package:16378560/2" technology="_" value="res"/>
 <part name="SUPPLY4" library="supply2" library_urn="urn:adsk.eagle:library:372" deviceset="GND" device=""/>
 <part name="H1" library="holes" library_urn="urn:adsk.eagle:library:237" deviceset="MOUNT-PAD-ROUND" device="3.0" package3d_urn="urn:adsk.eagle:package:14280/1"/>
@@
 <part name="SUPPLY5" library="supply2" library_urn="urn:adsk.eagle:library:372" deviceset="GND" device=""/>
 <part name="SUPPLY6" library="supply2" library_urn="urn:adsk.eagle:library:372" deviceset="GND" device=""/>
+<part name="U$2" library="Breakouts" deviceset="BMP388BREAKOUT" device=""/>
+<part name="SUPPLY7" library="supply2" library_urn="urn:adsk.eagle:library:372" deviceset="GND" device=""/>
+<part name="R1" library="rcl" library_urn="urn:adsk.eagle:library:334" deviceset="R-US_" device="0204/7" package3d_urn="urn:adsk.eagle:package:23498/2" value="10kΩ"/>
+<part name="X3" library="JST-XH Connectors" deviceset="JST-XH-02-PIN" device=""/>
 </parts>
 <sheets>
 <sheet>
 <plain>
-<text x="198.12" y="83.82" size="1.778" layer="91">double check these pins</text>
 </plain>
 <instances>
@@
 <attribute name="SHEET" x="230.505" y="5.08" size="2.54" layer="94"/>
 </instance>
-<instance part="U$1" gate="G$1" x="139.7" y="76.2" smashed="yes"/>
-<instance part="SUPPLY1" gate="GND" x="129.54" y="76.2" smashed="yes">
-<attribute name="VALUE" x="127.635" y="73.025" size="1.778" layer="96"/>
-</instance>
 <instance part="SUPPLY2" gate="GND" x="195.58" y="134.62" smashed="yes">
 <attribute name="VALUE" x="193.675" y="131.445" size="1.778" layer="96"/>
@@
 <attribute name="NAME" x="38.862" y="149.86" size="1.524" layer="95" rot="R90"/>
 </instance>
-<instance part="R1" gate="G$1" x="114.3" y="27.94" smashed="yes">
-<attribute name="NAME" x="114.3" y="30.48" size="1.778" layer="95" align="center"/>
-<attribute name="VALUE" x="114.3" y="25.4" size="1.778" layer="96" align="center"/>
-</instance>
-<instance part="R2" gate="G$1" x="93.98" y="27.94" smashed="yes">
-<attribute name="NAME" x="93.98" y="30.48" size="1.778" layer="95" align="center"/>
-<attribute name="VALUE" x="93.98" y="25.4" size="1.778" layer="96" align="center"/>
-</instance>
 <instance part="SUPPLY4" gate="GND" x="78.74" y="20.32" smashed="yes">
 <attribute name="VALUE" x="76.835" y="17.145" size="1.778" layer="96"/>
@@
 <instance part="SUPPLY6" gate="GND" x="208.28" y="38.1" smashed="yes">
 <attribute name="VALUE" x="206.375" y="34.925" size="1.778" layer="96"/>
+</instance>
+<instance part="U$2" gate="G$1" x="154.94" y="78.74" smashed="yes"/>
+<instance part="SUPPLY7" gate="GND" x="139.7" y="60.96" smashed="yes">
+<attribute name="VALUE" x="137.795" y="57.785" size="1.778" layer="96"/>
+</instance>
+<instance part="R1" gate="G$1" x="116.84" y="27.94" smashed="yes">
+<attribute name="NAME" x="113.03" y="29.4386" size="1.778" layer="95"/>
+<attribute name="VALUE" x="113.03" y="24.638" size="1.778" layer="96"/>
+</instance>
+<instance part="X3" gate="-2" x="86.36" y="35.56" smashed="yes">
+<attribute name="NAME" x="88.9" y="34.798" size="1.524" layer="95"/>
+</instance>
+<instance part="X3" gate="-1" x="86.36" y="38.1" smashed="yes">
+<attribute name="NAME" x="88.9" y="37.338" size="1.524" layer="95"/>
+<attribute name="VALUE" x="85.598" y="39.497" size="1.778" layer="96"/>
 </instance>
 </instances>
@@
 <net name="GPIO2" class="0">
 <segment>
-<wire x1="170.18" y1="81.28" x2="182.88" y2="81.28" width="0.1524" layer="91"/>
-<pinref part="U$1" gate="G$1" pin="INT"/>
-<label x="182.88" y="81.28" size="1.778" layer="95" xref="yes"/>
-</segment>
-<segment>
 <wire x1="35.56" y1="144.78" x2="35.56" y2="142.24" width="0.1524" layer="91"/>
 <label x="35.56" y="142.24" size="1.778" layer="95" rot="R270" xref="yes"/>
 <pinref part="X2" gate="-6" pin="S"/>
 </segment>
+<segment>
+<pinref part="U$2" gate="G$1" pin="INT"/>
+<wire x1="142.24" y1="71.12" x2="134.62" y2="71.12" width="0.1524" layer="91"/>
+<label x="134.62" y="71.12" size="1.778" layer="95" rot="MR0" xref="yes"/>
+</segment>
 </net>
 <net name="SDA" class="0">
@@
 </segment>
 <segment>
-<pinref part="U$1" gate="G$1" pin="SDI"/>
-<wire x1="170.18" y1="86.36" x2="175.26" y2="86.36" width="0.1524" layer="91"/>
-<label x="175.26" y="86.36" size="1.778" layer="95" xref="yes"/>
+<pinref part="U$2" gate="G$1" pin="SDA"/>
+<wire x1="142.24" y1="76.2" x2="134.62" y2="76.2" width="0.1524" layer="91"/>
+<label x="134.62" y="76.2" size="1.778" layer="95" rot="MR0" xref="yes"/>
 </segment>
 </net>
 <net name="SCL" class="0">
-<segment>
-<pinref part="U$1" gate="G$1" pin="SCL"/>
-<wire x1="170.18" y1="91.44" x2="182.88" y2="91.44" width="0.1524" layer="91"/>
-<label x="182.88" y="91.44" size="1.778" layer="95" xref="yes"/>
-</segment>
 <segment>
 <wire x1="134.62" y1="127" x2="124.46" y2="127" width="0.1524" layer="91"/>
@@
 <pinref part="X2" gate="-3" pin="S"/>
 </segment>
+<segment>
+<pinref part="U$2" gate="G$1" pin="SCL"/>
+<wire x1="142.24" y1="81.28" x2="134.62" y2="81.28" width="0.1524" layer="91"/>
+<label x="134.62" y="81.28" size="1.778" layer="95" rot="MR0" xref="yes"/>
+</segment>
 </net>
 <net name="GND" class="0">
-<segment>
-<pinref part="U$1" gate="G$1" pin="GND"/>
-<wire x1="134.62" y1="83.82" x2="129.54" y2="83.82" width="0.1524" layer="91"/>
-<wire x1="129.54" y1="83.82" x2="129.54" y2="78.74" width="0.1524" layer="91"/>
-<pinref part="SUPPLY1" gate="GND" pin="GND"/>
-</segment>
 <segment>
 <wire x1="73.66" y1="129.54" x2="73.66" y2="127" width="0.1524" layer="91"/>
@@
 </segment>
 <segment>
-<pinref part="R2" gate="G$1" pin="1"/>
-<wire x1="88.9" y1="27.94" x2="78.74" y2="27.94" width="0.1524" layer="91"/>
-<wire x1="78.74" y1="27.94" x2="78.74" y2="22.86" width="0.1524" layer="91"/>
 <pinref part="SUPPLY4" gate="GND" pin="GND"/>
+<wire x1="78.74" y1="22.86" x2="78.74" y2="38.1" width="0.1524" layer="91"/>
+<pinref part="X3" gate="-1" pin="S"/>
+<wire x1="78.74" y1="38.1" x2="83.82" y2="38.1" width="0.1524" layer="91"/>
 </segment>
 <segment>
@@
 <wire x1="83.82" y1="55.88" x2="83.82" y2="50.8" width="0.1524" layer="91"/>
 </segment>
+<segment>
+<pinref part="U$2" gate="G$1" pin="GND"/>
+<wire x1="142.24" y1="83.82" x2="139.7" y2="83.82" width="0.1524" layer="91"/>
+<wire x1="139.7" y1="83.82" x2="139.7" y2="63.5" width="0.1524" layer="91"/>
+<pinref part="SUPPLY7" gate="GND" pin="GND"/>
+</segment>
 </net>
 <net name="VBAT" class="0">
@@
 </segment>
 <segment>
-<pinref part="U$1" gate="G$1" pin="3VO"/>
-<wire x1="134.62" y1="86.36" x2="121.92" y2="86.36" width="0.1524" layer="91"/>
-<label x="121.92" y="86.36" size="1.778" layer="95" rot="R180" xref="yes"/>
+<pinref part="U$2" gate="G$1" pin="3VO"/>
+<wire x1="142.24" y1="86.36" x2="134.62" y2="86.36" width="0.1524" layer="91"/>
+<label x="134.62" y="86.36" size="1.778" layer="95" rot="MR0" xref="yes"/>
 </segment>
 <segment>
 <pinref part="R1" gate="G$1" pin="2"/>
-<wire x1="119.38" y1="27.94" x2="127" y2="27.94" width="0.1524" layer="91"/>
-<label x="127" y="27.94" size="1.778" layer="95" xref="yes"/>
+<wire x1="121.92" y1="27.94" x2="124.46" y2="27.94" width="0.1524" layer="91"/>
+<label x="124.46" y="27.94" size="1.778" layer="95" xref="yes"/>
 </segment>
 </net>
@@
 </segment>
 <segment>
+<wire x1="104.14" y1="27.94" x2="104.14" y2="38.1" width="0.1524" layer="91"/>
+<label x="104.14" y="38.1" size="1.778" layer="95" xref="yes"/>
+<pinref part="X3" gate="-2" pin="S"/>
+<wire x1="83.82" y1="35.56" x2="81.28" y2="35.56" width="0.1524" layer="91"/>
+<wire x1="81.28" y1="35.56" x2="81.28" y2="27.94" width="0.1524" layer="91"/>
+<wire x1="81.28" y1="27.94" x2="104.14" y2="27.94" width="0.1524" layer="91"/>
 <pinref part="R1" gate="G$1" pin="1"/>
-<pinref part="R2" gate="G$1" pin="2"/>
-<wire x1="109.22" y1="27.94" x2="104.14" y2="27.94" width="0.1524" layer="91"/>
-<wire x1="104.14" y1="27.94" x2="99.06" y2="27.94" width="0.1524" layer="91"/>
-<wire x1="104.14" y1="27.94" x2="104.14" y2="38.1" width="0.1524" layer="91"/>
+<wire x1="111.76" y1="27.94" x2="104.14" y2="27.94" width="0.1524" layer="91"/>
 <junction x="104.14" y="27.94"/>
-<label x="104.14" y="38.1" size="1.778" layer="95" xref="yes"/>
-</segment>
-</net>
+</segment>
+</net>
